Commit message: Refine articulated assets and add reference comparisons

File: assets/batch5_collision_urdf_textured/100520/100520.urdf (robot description, URDF)
Before this commit: robot 100520, 5 links, 4 joints
Joints:
- joint rear_frame_fold: limit lower=0 upper=0.0349065850399 effort=1 velocity=1 -> lower=-1.047197551197 upper=0.0349065850399 effort=1 velocity=1
- joint seat_fold: limit lower=-0.349065850399 upper=0 effort=1 velocity=1 -> lower=-1.570796326795 upper=0 effort=1 velocity=1
